Commit message: Test Manager works for gripper, caster. Viewer displays state of all tests

File: life_test/caster_life_test/caster.urdf.xacro (robot description, xacro)
@@ -1,9 +1,37 @@
 <?xml version="1.0"?>
-<robot>
+<robot name="caster" >
   <include filename="$(find pr2_defs)/calibration/default_cal.xml" />
   <include filename="$(find pr2_defs)/defs/base/base_defs.urdf.xacro" />
   <include filename="$(find pr2_defs)/defs/materials.urdf.xacro" />
-  <pr2_caster suffix="fl" parent="world">
+  <pr2_caster suffix="fl" parent="base_link" >
     <origin xyz="0 0 0" rpy="0 0 0" />
   </pr2_caster>
+  <!-- Solid Base for visualizer -->
+  <joint name="base_joint" type="fixed">
+    <parent link="world" />
+    <origin xyz="0 0 0" rpy="0 0 0" />
+    <child link="base_link" />
+  </joint>
+  <link name="base_link">
+    <inertial>
+      <mass value="1000" />
+      <origin xyz=" 0 0 0 " />
+      <inertia ixx="1000"  ixy="0"  ixz="0" iyy="1000" iyz="0" izz="1000" />
+    </inertial>
+    <visual>
+      <origin xyz="0 0 -1" rpy="0 0 0 " />
+      <geometry name="pr2_base_mesh_file">
+        <mesh scale="20 20 0.01" />
+      </geometry>
+    </visual>
+    <collision>
+      <origin xyz="0 0 -1" rpy="0.0 0.0 0.0 " />
+      <geometry name="base_collision_geom">
+        <box size="20 20 0.01" />
+      </geometry>
+    </collision>
+  </link>
+  <gazebo reference="base_link" >
+    <material>Gazebo/White</material>
+  </gazebo>
 </robot>
