Commit message: Hokuyo range test works. Gripper drop test works with LED check

File: qualification/tests/caster_test/caster.urdf.xacro (robot description, xacro)
@@ -1,25 +1,24 @@
 <?xml version="1.0"?>
-<robot name="test_caster">
+<robot name="caster" >
   <include filename="$(find pr2_defs)/calibration/default_cal.xml" />
-  <include filename="$(find pr2_defs)/defs/base_defs.xml" />
-<pr2_caster_alpha2 suffix="fl" parent="base_link" ref_position="0.0" >
-      <origin xyz="0 0 0" rpy="0 0 0" />
-</pr2_caster_alpha2>
+  <include filename="$(find pr2_defs)/defs/base/base_defs.urdf.xacro" />
+  <include filename="$(find pr2_defs)/defs/materials.urdf.xacro" />
+  <pr2_caster suffix="fl" parent="base_link" ref_position="0.0" >
+    <origin xyz="0 0 0" rpy="0 0 0" />
+  </pr2_caster>
   <!-- Solid Base for visualizer -->
-  <joint name="base_joint" type="planar" />
+  <joint name="base_joint" type="fixed">
+    <parent link="world" />
+    <origin xyz="0 0 0" rpy="0 0 0" />
+    <child link="base_link" />
+  </joint>
   <link name="base_link">
-    <parent name=" world" />
-    <origin xyz=" 0 0 1 " rpy=" 0 0 0" />
-    <joint name="base_joint" />
     <inertial>
       <mass value="1000" />
-      <com xyz=" 0 0 0 " />
+      <origin xyz=" 0 0 0 " />
       <inertia ixx="1000"  ixy="0"  ixz="0" iyy="1000" iyz="0" izz="1000" />
     </inertial>
     <visual>
       <origin xyz="0 0 -1" rpy="0 0 0 " />
-      <map name="gazebo_material" flag="gazebo">
-        <elem key="material">Gazebo/White</elem>
-      </map>
       <geometry name="pr2_base_mesh_file">
         <mesh scale="20 20 0.01" />
@@ -33,3 +32,6 @@
     </collision>
   </link>
+  <gazebo reference="base_link" >
+    <material>Gazebo/White</material>
+  </gazebo>
 </robot>

File: qualification/tests/caster_test/caster_alpha2.urdf.xacro (robot description, xacro)
@@ -1,25 +1,24 @@
 <?xml version="1.0"?>
-<robot name="test_caster">
+<robot name="caster" >
   <include filename="$(find pr2_defs)/calibration/default_cal.xml" />
-  <include filename="$(find pr2_defs)/defs/base_defs.xml" />
-<pr2_caster suffix="fl" parent="base_link">
-      <origin xyz="0 0 0" rpy="0 0 0" />
-</pr2_caster>
+  <include filename="$(find pr2_defs)/defs/base/alpha2_base_defs.urdf.xacro" />
+  <include filename="$(find pr2_defs)/defs/materials.urdf.xacro" />
+  <pr2_caster_alpha2 suffix="fl" parent="base_link" ref_position="0.0" >
+    <origin xyz="0 0 0" rpy="0 0 0" />
+  </pr2_caster_alpha2>
   <!-- Solid Base for visualizer -->
-  <joint name="base_joint" type="planar" />
+  <joint name="base_joint" type="fixed">
+    <parent link="world" />
+    <origin xyz="0 0 0" rpy="0 0 0" />
+    <child link="base_link" />
+  </joint>
   <link name="base_link">
-    <parent name="world" />
-    <origin xyz=" 0 0 1 " rpy=" 0 0 0" />
-    <joint name="base_joint" />
     <inertial>
       <mass value="1000" />
-      <com xyz=" 0 0 0 " />
+      <origin xyz=" 0 0 0 " />
       <inertia ixx="1000"  ixy="0"  ixz="0" iyy="1000" iyz="0" izz="1000" />
     </inertial>
     <visual>
       <origin xyz="0 0 -1" rpy="0 0 0 " />
-      <map name="gazebo_material" flag="gazebo">
-        <elem key="material">Gazebo/White</elem>
-      </map>
       <geometry name="pr2_base_mesh_file">
         <mesh scale="20 20 0.01" />
@@ -33,3 +32,6 @@
     </collision>
   </link>
+  <gazebo reference="base_link" >
+    <material>Gazebo/White</material>
+  </gazebo>
 </robot>
