Commit message: Changing all URDF files to new pr2_description package. Gripper, Caster, Wrist all tested on HW

File: qualification/tests/caster_test/caster_motor.urdf.xacro (robot description, xacro)
@@ -1,5 +1,5 @@
 <?xml version="1.0"?>
-<robot name="motor">
-  <joint name="motor_joint" type="continuous">
+<robot name="caster_motor">
+  <joint name="caster_motor_joint" type="continuous">
     <axis xyz="0 1 0" />
     <limit effort="100" velocity="100"/>
@@ -8,7 +8,7 @@
     <origin xyz="0 0 0" rpy="0 0 0" />
     <parent link="world"/>
-    <child link="motor_link"/>
+    <child link="caster_motor_link"/>
   </joint>
-  <link name="motor_link">
+  <link name="caster_motor_link">
     <inertial>
       <mass value="1" />
@@ -19,7 +19,7 @@
   </link>
   <!-- Transmission uses fl_caster_l_wheel_motor -->
-  <transmission type="SimpleTransmission" name="motor_trans">
+  <transmission type="SimpleTransmission" name="caster_motor_trans">
     <actuator name="fl_caster_l_wheel_motor" />
-    <joint name="motor_joint" />
+    <joint name="caster_motor_joint" />
     <mechanicalReduction>${624/35}</mechanicalReduction>
   </transmission>

File: qualification/tests/full_arm_test/full_arm.urdf.xacro (robot description, xacro)
@@ -1,4 +1,4 @@
 <?xml version="1.0"?>
-<robot name="test_gripper"
+<robot name="pr2_arm"
        xmlns:sensor="http://playerstage.sourceforge.net/gazebo/xmlschema/#sensor"
        xmlns:controller="http://playerstage.sourceforge.net/gazebo/xmlschema/#controller"
@@ -7,16 +7,26 @@
   <include filename="$(find pr2_description)/urdf/common.xacro" />
   <include filename="$(find pr2_description)/urdf/materials.urdf.xacro" />
+  <!-- PR2 Arm -->
+  <include filename="$(find pr2_description)/urdf/shoulder_v0/shoulder.urdf.xacro" />
+  <include filename="$(find pr2_description)/urdf/upper_arm_v0/upper_arm.urdf.xacro" />
+  <include filename="$(find pr2_description)/urdf/forearm_v0/forearm.urdf.xacro" />
+  <!-- PR2 gripper -->
   <include filename="$(find pr2_description)/urdf/gripper_v0/gripper.urdf.xacro" />
-  <xacro:pr2_gripper_v0 side="r" parent="base_link"
-                        screw_reduction="${4.0/1000.0}"
-                        gear_ratio="${(729.0/25.0)*(22.0/16.0)}"
-                        theta0="${3.6029*M_PI/180.0}"
-                        phi0="${29.7089*M_PI/180.0}"
-                        t0="${-0.1914/1000.0}"
-                        L0="${37.5528/1000.0}"
-                        h="${0.0/1000.0}"
-                        a="${68.3698/1000.0}"
-                        b="${43.3849/1000.0}"
-                        r="${91.5/1000.0}" >
+  <xacro:pr2_shoulder_v0 side="r" reflect="-1" parent="base_link">
+    <origin xyz="0.0 -0.188 0.0" rpy="0 0 0" />
+  </xacro:pr2_shoulder_v0>
+  <xacro:pr2_upper_arm_v0 side="r" reflect="-1" parent="r_upper_arm_roll_link"/>
+  <xacro:pr2_forearm_v0 side="r" reflect="-1" parent="r_forearm_roll_link"/>
+  <xacro:pr2_gripper_v0 side="r" parent="r_wrist_roll_link"
+               screw_reduction="${4.0/1000.0}"
+               gear_ratio="${(729.0/25.0)*(22.0/16.0)}"
+               theta0="${3.6029*M_PI/180.0}"
+               phi0="${29.7089*M_PI/180.0}"
+               t0="${-0.1914/1000.0}"
+               L0="${37.5528/1000.0}"
+               h="${0.0/1000.0}"
+               a="${68.3698/1000.0}"
+               b="${43.3849/1000.0}"
+               r="${91.5/1000.0}" >
     <origin xyz="0 0 0" rpy="0 0 0" />
   </xacro:pr2_gripper_v0>

File: qualification/tests/head_test/head.urdf.xacro (robot description, xacro)
@@ -6,6 +6,6 @@
        xmlns:xacro="http://ros.org/wiki/xacro">
   <include filename="$(find pr2_description)/urdf/common.xacro" />
+  <include filename="$(find pr2_description)/urdf/materials.urdf.xacro" />
   <include filename="$(find pr2_description)/urdf/head_v0/head.urdf.xacro" />
-  <include filename="$(find pr2_description)/urdf/materials.urdf.xacro" />
   <xacro:pr2_head_v0 name="head" parent="base_link">
     <origin xyz="0 0 0" rpy="0 0 0" />
@@ -26,5 +26,5 @@
       <origin xyz="0 0 0" rpy="0 0 0 " />
       <geometry name="pr2_base_mesh_file">
-        <mesh scale="20 20 0.01" />
+        <box size="1 1 1" />
       </geometry>
     </visual>

File: qualification/tests/shoulder_test/shoulder.urdf.xacro (robot description, xacro)
@@ -1,4 +1,4 @@
 <?xml version="1.0"?>
-<robot name="caster"
+<robot name="shoulder"
        xmlns:sensor="http://playerstage.sourceforge.net/gazebo/xmlschema/#sensor"
        xmlns:controller="http://playerstage.sourceforge.net/gazebo/xmlschema/#controller"
@@ -7,8 +7,8 @@
   <include filename="$(find pr2_description)/urdf/common.xacro" />
   <include filename="$(find pr2_description)/urdf/materials.urdf.xacro" />
-  <include filename="$(find pr2_description)/urdf/base_v0/base.urdf.xacro" />
-  <xacro:pr2_caster_v0 suffix="fl" parent="base_link" ref_position="0.0" >
+  <include filename="$(find pr2_description)/urdf/shoulder_v0/shoulder.urdf.xacro" />
+  <xacro:pr2_shoulder_v0 side="r" reflect="-1" parent="base_link">
     <origin xyz="0 0 0" rpy="0 0 0" />
-  </xacro:pr2_caster_v0>
+  </xacro:pr2_shoulder_v0>
   <!-- Solid Base for visualizer -->
   <joint name="base_joint" type="fixed">
@@ -21,16 +21,16 @@
       <mass value="1000" />
       <origin xyz=" 0 0 0 " />
-      <inertia ixx="1000"  ixy="0"  ixz="0" iyy="1000" iyz="0" izz="1000" />
+      <inertia ixx="1000" ixy="0" ixz="0" iyy="1000" iyz="0" izz="1000" />
     </inertial>
     <visual>
-      <origin xyz="0 0 -1" rpy="0 0 0 " />
+      <origin xyz="0 0 0" rpy="0 0 0 " />
       <geometry name="pr2_base_mesh_file">
-        <box size="20 20 0.01" />
+        <box size="1 1 1" />
       </geometry>
     </visual>
     <collision>
-      <origin xyz="0 0 -1" rpy="0.0 0.0 0.0 " />
+      <origin xyz="0 0 0" rpy="0.0 0.0 0.0 " />
       <geometry name="base_collision_geom">
-        <box size="20 20 0.01" />
+        <box size="1 1 1" />
       </geometry>
     </collision>

File: qualification/tests/torso_lift_test/torso.urdf.xacro (robot description, xacro)
@@ -1,4 +1,4 @@
 <?xml version="1.0"?>
-<robot name="caster"
+<robot name="torso"
        xmlns:sensor="http://playerstage.sourceforge.net/gazebo/xmlschema/#sensor"
        xmlns:controller="http://playerstage.sourceforge.net/gazebo/xmlschema/#controller"
@@ -7,8 +7,8 @@
   <include filename="$(find pr2_description)/urdf/common.xacro" />
   <include filename="$(find pr2_description)/urdf/materials.urdf.xacro" />
-  <include filename="$(find pr2_description)/urdf/base_v0/base.urdf.xacro" />
-  <xacro:pr2_caster_v0 suffix="fl" parent="base_link" ref_position="0.0" >
+  <include filename="$(find pr2_description)/urdf/torso_v0/torso.urdf.xacro" />
+  <xacro:pr2_torso_v0 name="torso" parent="base_link">
     <origin xyz="0 0 0" rpy="0 0 0" />
-  </xacro:pr2_caster_v0>
+  </xacro:pr2_torso_v0>
   <!-- Solid Base for visualizer -->
   <joint name="base_joint" type="fixed">
@@ -21,16 +21,16 @@
       <mass value="1000" />
       <origin xyz=" 0 0 0 " />
-      <inertia ixx="1000"  ixy="0"  ixz="0" iyy="1000" iyz="0" izz="1000" />
+      <inertia ixx="1000" ixy="0" ixz="0" iyy="1000" iyz="0" izz="1000" />
     </inertial>
     <visual>
-      <origin xyz="0 0 -1" rpy="0 0 0 " />
+      <origin xyz="0 0 0" rpy="0 0 0 " />
       <geometry name="pr2_base_mesh_file">
-        <box size="20 20 0.01" />
+        <box size="1 1 1" />
       </geometry>
     </visual>
     <collision>
-      <origin xyz="0 0 -1" rpy="0.0 0.0 0.0 " />
+      <origin xyz="0 0 0" rpy="0.0 0.0 0.0 " />
       <geometry name="base_collision_geom">
-        <box size="20 20 0.01" />
+        <box size="1 1 1" />
       </geometry>
     </collision>

File: qualification/tests/upperarm_test/upperarm.urdf.xacro (robot description, xacro)
@@ -1,4 +1,4 @@
 <?xml version="1.0"?>
-<robot name="caster"
+<robot name="pr2_upper_arm"
        xmlns:sensor="http://playerstage.sourceforge.net/gazebo/xmlschema/#sensor"
        xmlns:controller="http://playerstage.sourceforge.net/gazebo/xmlschema/#controller"
@@ -7,8 +7,8 @@
   <include filename="$(find pr2_description)/urdf/common.xacro" />
   <include filename="$(find pr2_description)/urdf/materials.urdf.xacro" />
-  <include filename="$(find pr2_description)/urdf/base_v0/base.urdf.xacro" />
-  <xacro:pr2_caster_v0 suffix="fl" parent="base_link" ref_position="0.0" >
+  <include filename="$(find pr2_description)/urdf/upper_arm_v0/upper_arm.urdf.xacro" />
+  <xacro:pr2_upper_arm_v0 side="r" reflect="-1" parent="base_link">
     <origin xyz="0 0 0" rpy="0 0 0" />
-  </xacro:pr2_caster_v0>
+  </xacro:pr2_upper_arm_v0>
   <!-- Solid Base for visualizer -->
   <joint name="base_joint" type="fixed">
@@ -21,16 +21,16 @@
       <mass value="1000" />
       <origin xyz=" 0 0 0 " />
-      <inertia ixx="1000"  ixy="0"  ixz="0" iyy="1000" iyz="0" izz="1000" />
+      <inertia ixx="1000" ixy="0" ixz="0" iyy="1000" iyz="0" izz="1000" />
     </inertial>
     <visual>
-      <origin xyz="0 0 -1" rpy="0 0 0 " />
+      <origin xyz="0 0 0" rpy="0 0 0 " />
       <geometry name="pr2_base_mesh_file">
-        <box size="20 20 0.01" />
+        <box size="1 1 1" />
       </geometry>
     </visual>
     <collision>
-      <origin xyz="0 0 -1" rpy="0.0 0.0 0.0 " />
+      <origin xyz="0 0 0" rpy="0.0 0.0 0.0 " />
       <geometry name="base_collision_geom">
-        <box size="20 20 0.01" />
+        <box size="1 1 1" />
       </geometry>
     </collision>

File: qualification/tests/wrist_test/wrist.urdf.xacro (robot description, xacro)
@@ -1,4 +1,4 @@
 <?xml version="1.0"?>
-<robot name="caster"
+<robot name="forearm"
        xmlns:sensor="http://playerstage.sourceforge.net/gazebo/xmlschema/#sensor"
        xmlns:controller="http://playerstage.sourceforge.net/gazebo/xmlschema/#controller"
@@ -7,8 +7,8 @@
   <include filename="$(find pr2_description)/urdf/common.xacro" />
   <include filename="$(find pr2_description)/urdf/materials.urdf.xacro" />
-  <include filename="$(find pr2_description)/urdf/base_v0/base.urdf.xacro" />
-  <xacro:pr2_caster_v0 suffix="fl" parent="base_link" ref_position="0.0" >
+  <include filename="$(find pr2_description)/urdf/forearm_v0/forearm.urdf.xacro" />
+  <xacro:pr2_forearm_v0 side="r" reflect="-1" parent="base_link">
     <origin xyz="0 0 0" rpy="0 0 0" />
-  </xacro:pr2_caster_v0>
+  </xacro:pr2_forearm_v0>
   <!-- Solid Base for visualizer -->
   <joint name="base_joint" type="fixed">
@@ -21,16 +21,16 @@
       <mass value="1000" />
       <origin xyz=" 0 0 0 " />
-      <inertia ixx="1000"  ixy="0"  ixz="0" iyy="1000" iyz="0" izz="1000" />
+      <inertia ixx="1000" ixy="0" ixz="0" iyy="1000" iyz="0" izz="1000" />
     </inertial>
     <visual>
-      <origin xyz="0 0 -1" rpy="0 0 0 " />
+      <origin xyz="0 0 0" rpy="0 0 0 " />
       <geometry name="pr2_base_mesh_file">
-        <box size="20 20 0.01" />
+        <box size="1 1 1" />
       </geometry>
     </visual>
     <collision>
-      <origin xyz="0 0 -1" rpy="0.0 0.0 0.0 " />
+      <origin xyz="0 0 0" rpy="0.0 0.0 0.0 " />
       <geometry name="base_collision_geom">
-        <box size="20 20 0.01" />
+        <box size="1 1 1" />
       </geometry>
     </collision>
