Commit message: Gripper life test working with corrected transmission

File: life_test/gripper_life_test/gripper.urdf.xacro (robot description, xacro)
@@ -1,8 +1,17 @@
 <?xml version="1.0"?>
-<robot name="gripper">
+<robot name="test_gripper">
   <include filename="$(find pr2_defs)/calibration/default_cal.xml" />
-  <include filename="$(find pr2_defs)/defs/gripper/gripper_defs.urdf.xacro" />
+  <include filename="$(find pr2_defs)/defs/gripper_beta/gripper_defs.urdf.xacro" />
   <include filename="$(find pr2_defs)/defs/materials.urdf.xacro" />
-  <pr2_gripper side="r" parent="base_link" screw_reduction="${4.0/1000.0}" gear_ratio="${29.16*22.0/16.0*0.9}" >
+  <pr2_gripper side="r" parent="base_link" screw_reduction="${4.0/1000.0}"
+               gear_ratio="${(729.0/25.0)*(22.0/16.0)}"
+               theta0="${3.6029*M_PI/180.0}"
+               phi0="${29.7089*M_PI/180.0}"
+               t0="${-0.1914/1000.0}"
+               L0="${37.5528/1000.0}"
+               h="${0.0/1000.0}"
+               a="${68.3698/1000.0}"
+               b="${43.3849/1000.0}"
+               r="${91.5/1000.0}" >
     <origin xyz="0 0 0" rpy="0 0 0" />
   </pr2_gripper>
@@ -10,5 +19,5 @@
   <joint name="base_joint" type="fixed">
     <parent link="world" />
-    <origin xyz="0 0 1" rpy="0 0 0" />
+    <origin xyz="0 0 0" rpy="0 0 0" />
     <child link="base_link" />
   </joint>
@@ -17,8 +26,8 @@
       <mass value="1000" />
       <origin xyz=" 0 0 0 " />
-      <inertia ixx="1000"  ixy="0"  ixz="0" iyy="1000" iyz="0" izz="1000" />
+      <inertia ixx="1000" ixy="0" ixz="0" iyy="1000" iyz="0" izz="1000" />
     </inertial>
     <visual>
-      <origin xyz="0 0 -1" rpy="0 0 0 " />
+      <origin xyz="0 0 0" rpy="0 0 0 " />
       <geometry name="pr2_base_mesh_file">
         <mesh scale="20 20 0.01" />
@@ -26,7 +35,7 @@
     </visual>
     <collision>
-      <origin xyz="0 0 -1" rpy="0.0 0.0 0.0 " />
+      <origin xyz="0 0 0" rpy="0.0 0.0 0.0 " />
       <geometry name="base_collision_geom">
-        <box size="20 20 0.01" />
+        <box size="1 1 1" />
       </geometry>
     </collision>
