Commit message: Corrections to prosilica test, head test works with new defs on HW

File: qualification/tests/head_test/head.urdf.xacro (robot description, xacro)
@@ -26,5 +26,5 @@
       <origin xyz="0 0 0" rpy="0 0 0 " />
       <geometry name="pr2_base_mesh_file">
-        <box size="1 1 1" />
+        <box size=".01 .01 .01" />
       </geometry>
     </visual>
@@ -32,5 +32,5 @@
       <origin xyz="0 0 0" rpy="0.0 0.0 0.0 " />
       <geometry name="base_collision_geom">
-        <box size="1 1 1" />
+        <box size=".01 .01 .01" />
       </geometry>
     </collision>
