Commit message: Laser tilt test tested for alpha prototype, still needs drop test

File: qualification/tests/head_test/head_tilt_motor.urdf.xacro (robot description, xacro)
@@ -18,5 +18,5 @@
     </inertial>
   </link>
-  <!-- Transmission uses head_tilt_motor -->
+  <!-- Transmission uses fl_caster_l_wheel_motor -->
   <transmission type="SimpleTransmission" name="head_tilt_motor_trans">
     <actuator name="head_tilt_motor" />

File: qualification/tests/laser_tilt_test/laser_tilt_motor.urdf.xacro (robot description, xacro)
@@ -1,10 +1,6 @@
 <?xml version="1.0"?>
-<robot name="tilting_laser"
-       xmlns:sensor="http://playerstage.sourceforge.net/gazebo/xmlschema/#sensor"
-       xmlns:controller="http://playerstage.sourceforge.net/gazebo/xmlschema/#controller"
-       xmlns:interface="http://playerstage.sourceforge.net/gazebo/xmlschema/#interface"
-       xmlns:xacro="http://ros.org/wiki/xacro">
+<robot name="tilting_laser">
   <joint name="laser_tilt_motor_joint" type="continuous">
-    <axis xyz="0 1 0" />
+    <axis xyz="0 0 1" />
     <limit effort="100" velocity="100"/>
     <safety_controller k_velocity="10" />
@@ -24,5 +20,5 @@
   <!-- Transmission uses laser_tilt_motor -->
   <transmission type="SimpleTransmission" name="laser_tilt_motor_trans">
-    <actuator name="laser_tilt_motor" />
+    <actuator name="laser_tilt_mount_motor" />
     <joint name="laser_tilt_motor_joint" />
     <mechanicalReduction>1</mechanicalReduction>

Commit message: Head tilt test on first Beta unit, caster hub test added

File: qualification/tests/head_test/head_tilt_motor.urdf.xacro (robot description, xacro)
@@ -10,14 +10,7 @@
     <child link="head_tilt_motor_link"/>
   </joint>
-  <link name="head_tilt_motor_link">
-    <inertial>
-      <mass value="1" />
-      <origin xyz=" 0 0 0 " />
-      <inertia  ixx="1.0" ixy="0.0" ixz="0.0"
-                iyy="1.0" iyz="0.0" izz="1.0" />
-    </inertial>
-  </link>
-  <!-- Transmission uses fl_caster_l_wheel_motor -->
-  <transmission type="SimpleTransmission" name="head_tilt_motor_trans">
+  <link name="head_tilt_motor_link" />
+  <transmission type="SimpleTransmission"
+                name="head_tilt_motor_trans">
     <actuator name="head_tilt_motor" />
     <joint name="head_tilt_motor_joint" />
