Commit message: Changing FA roll motor URDF for correct joint/motor names

File: pr2_component_descriptions/robot_motors/forearm_roll_motor.urdf.xacro (robot description, xacro)
@@ -1,5 +1,5 @@
 <?xml version="1.0"?>
-<robot name="forearm_roll_motor">
-  <joint name="forearm_roll_motor_joint" type="continuous">
+<robot name="r_forearm_roll_motor">
+  <joint name="r_forearm_roll_motor_joint" type="continuous">
     <axis xyz="0 0 1" />
     <limit effort="100" velocity="100"/>
@@ -8,7 +8,7 @@
     <origin xyz="0 0 0" rpy="0 0 0" />
     <parent link="world"/>
-    <child link="forearm_roll_motor_link"/>
+    <child link="r_forearm_roll_motor_link"/>
   </joint>
-  <link name="forearm_roll_motor_link">
+  <link name="r_forearm_roll_motor_link">
     <inertial>
       <mass value="1" />
@@ -19,7 +19,7 @@
   </link>
   <!-- Transmission uses forearm_roll_motor -->
-  <transmission type="SimpleTransmission" name="forearm_roll_motor_trans">
-    <actuator name="forearm_roll_motor" />
-    <joint name="forearm_roll_motor_joint" />
+  <transmission type="SimpleTransmission" name="r_forearm_roll_motor_trans">
+    <actuator name="r_forearm_roll_motor" />
+    <joint name="r_forearm_roll_motor_joint" />
     <mechanicalReduction>1</mechanicalReduction>
   </transmission>
