Commit message: Added invent parameters to qualification system, so they can be machine readable.

File: pr2_component_descriptions/robot_motors/caster_motor.urdf.xacro (robot description, xacro)
@@ -10,5 +10,5 @@
     <child link="caster_motor_link"/>
   </joint>
-  <link name="caster_motor_link">
+  <link name="caster_motor_link" >
     <inertial>
       <mass value="1" />
