Commit message: Addign shoulder lift motor URDF

File: pr2_component_descriptions/robot_motors/shoulder_lift_motor.urdf.xacro (robot description, xacro)
@@ -1,5 +1,5 @@
 <?xml version="1.0"?>
-<robot name="elbow_flex_motor">
-  <joint name="elbow_flex_motor_joint" type="continuous">
+<robot name="shoulder_lift_motor">
+  <joint name="shoulder_lift_motor_joint" type="continuous">
     <axis xyz="0 0 1" />
     <limit effort="100" velocity="100"/>
@@ -8,7 +8,7 @@
     <origin xyz="0 0 0" rpy="0 0 0" />
     <parent link="world"/>
-    <child link="elbow_flex_motor_link"/>
+    <child link="shoulder_lift_motor_link"/>
   </joint>
-  <link name="elbow_flex_motor_link">
+  <link name="shoulder_lift_motor_link">
     <inertial>
       <mass value="1" />
@@ -18,8 +18,8 @@
     </inertial>
   </link>
-  <!-- Transmission uses elbow_flex_motor -->
-  <transmission type="SimpleTransmission" name="elbow_flex_motor_trans">
-    <actuator name="r_elbow_flex_motor" />
-    <joint name="elbow_flex_motor_joint" />
+  <!-- Transmission uses shoulder_lift_motor -->
+  <transmission type="SimpleTransmission" name="shoulder_lift_motor_trans">
+    <actuator name="r_shoulder_lift_motor" />
+    <joint name="shoulder_lift_motor_joint" />
     <!-- This is clearly wrong. Need exact number -->
     <mechanicalReduction>${13/3}</mechanicalReduction>
