Commit message: UA, FA defs with dummy FA, gripper

File: pr2_component_descriptions/robots/upperarm_wrist.urdf.xacro (robot description, xacro)
@@ -8,11 +8,37 @@
   <include filename="$(find pr2_description)/urdf/materials.urdf.xacro" />
   <include filename="$(find pr2_description)/urdf/upper_arm_v0/upper_arm.urdf.xacro" />
-  <include filename="$(find pr2_description)/urdf/forearm_v0/forearm.urdf.xacro" />
   <include filename="$(find pr2_component_descriptions)/urdf/base_link.urdf.xacro" />
   <xacro:pr2_upper_arm_v0 side="r" reflect="-1" parent="base_link">
     <origin xyz="0 0 0" rpy="0 0 0" />
   </xacro:pr2_upper_arm_v0>
-    <xacro:pr2_forearm_v0 side="r" reflect="-1" parent="r_forearm_roll_link">
+    <!-- Dummy FA used in burn in test -->
+  <joint name="r_dummy_forearm_joint" type="continuous">
+    <axis xyz="0 1 0" />
+    <limit effort="0" velocity="100"/>
+    <safety_controller k_velocity="10" />
+    <dynamics damping="0.0" friction="0.0" />
     <origin xyz="0 0 0" rpy="0 0 0" />
-  </xacro:pr2_forearm_v0>
+    <parent link="r_forearm_roll_link"/>
+    <child link="r_dummy_forearm_link"/>
+  </joint>
+  <link name="r_dummy_forearm_link">
+    <inertial>
+      <mass value="1" />
+      <origin xyz=" 0 0 0 " />
+      <inertia  ixx="1.0" ixy="0.0" ixz="0.0"
+                iyy="1.0" iyz="0.0" izz="1.0" />
+    </inertial>
+    <visual>
+      <origin xyz="0.10 0 0" rpy="0 0 0" />
+      <geometry>
+	<box size="0.30 0.10 0.10" />
+      </geometry>
+    </visual>
+  </link>
+  <!-- Transmission uses r_gripper_motor -->
+  <transmission type="SimpleTransmission" name="r_dummy_forearm_trans">
+    <actuator name="r_wrist_l_motor" />
+    <joint name="r_dummy_forearm_joint" />
+    <mechanicalReduction>1</mechanicalReduction>
+  </transmission>
 </robot>

File: pr2_component_descriptions/robots/wrist_gripper.urdf.xacro (robot description, xacro)
@@ -18,5 +18,5 @@
   <joint name="r_gripper_fake_joint" type="continuous">
     <axis xyz="0 1 0" />
-    <limit effort="100" velocity="100"/>
+    <limit effort="0" velocity="100"/>
     <safety_controller k_velocity="10" />
     <dynamics damping="0.0" friction="0.0" />
@@ -32,4 +32,10 @@
                 iyy="1.0" iyz="0.0" izz="1.0" />
     </inertial>
+    <visual>
+      <origin xyz="0 0 0" rpy="0 0 0" />
+      <geometry>
+	<box size="0.12 0.10 0.12" />
+      </geometry>
+    </visual>
   </link>
   <!-- Transmission uses r_gripper_motor -->
