Commit message: Changed gripper def to fake gripper for wrist burn in test

File: pr2_component_descriptions/robots/wrist_gripper.urdf.xacro (robot description, xacro)
@@ -15,16 +15,27 @@
     <origin xyz="0 0 0" rpy="0 0 0" />
   </xacro:pr2_forearm_v0>
-  <xacro:pr2_gripper_v0 side="r" parent="r_wrist_roll_link"
-                        screw_reduction="${4.0/1000.0}"
-                        gear_ratio="${(729.0/25.0)*(22.0/16.0)}"
-                        theta0="${3.6029*M_PI/180.0}"
-                        phi0="${29.7089*M_PI/180.0}"
-                        t0="${-0.1914/1000.0}"
-                        L0="${37.5528/1000.0}"
-                        h="${0.0/1000.0}"
-                        a="${68.3698/1000.0}"
-                        b="${43.3849/1000.0}"
-                        r="${91.5/1000.0}" >
+  <!-- Dummy gripper used in burn in test -->
+  <joint name="r_gripper_fake_joint" type="continuous">
+    <axis xyz="0 1 0" />
+    <limit effort="100" velocity="100"/>
+    <safety_controller k_velocity="10" />
+    <dynamics damping="0.0" friction="0.0" />
     <origin xyz="0 0 0" rpy="0 0 0" />
-  </xacro:pr2_gripper_v0>
+    <parent link="r_wrist_roll_link"/>
+    <child link="r_gripper_fake_link"/>
+  </joint>
+  <link name="r_gripper_fake_link">
+    <inertial>
+      <mass value="1" />
+      <origin xyz=" 0 0 0 " />
+      <inertia  ixx="1.0" ixy="0.0" ixz="0.0"
+                iyy="1.0" iyz="0.0" izz="1.0" />
+    </inertial>
+  </link>
+  <!-- Transmission uses r_gripper_motor -->
+  <transmission type="SimpleTransmission" name="r_gripper_fake_trans">
+    <actuator name="r_gripper_motor" />
+    <joint name="r_gripper_fake_joint" />
+    <mechanicalReduction>1</mechanicalReduction>
+  </transmission>
 </robot>

Commit message: Correcting shape of dummy gripper in visualizer

File: pr2_component_descriptions/robots/wrist_gripper.urdf.xacro (robot description, xacro)
@@ -33,7 +33,7 @@
     </inertial>
     <visual>
-      <origin xyz="0 0 0" rpy="0 0 0" />
+      <origin xyz="0.06 0 0" rpy="0 0 0" />
       <geometry>
-	<box size="0.12 0.10 0.12" />
+	<box size="0.06 0.06 0.05" />
       </geometry>
     </visual>
