Commit message: fictitous world link deprecated. raise forearm fixture 2m from ground.

File: pr2_component_descriptions/robots/wrist.urdf.xacro (robot description, xacro)
@@ -12,5 +12,5 @@
   <include filename="$(find pr2_description)/gazebo/gazebo.urdf.xacro" />
   <xacro:pr2_forearm_v0 side="r" reflect="-1" parent="base_link">
-    <origin xyz="0 0 0" rpy="0 0 0" />
+    <origin xyz="0 0 2" rpy="0 0 0" />
   </xacro:pr2_forearm_v0>
 </robot>

File: pr2_component_descriptions/urdf/base_link.urdf.xacro (robot description, xacro)
@@ -3,25 +3,20 @@
 <!-- Including this file will include the link, no macro needed -->
 <!-- include filename="$(find pr2_component_description)/urdf/base_link.urdf.xacro" -->
-<robot>
-  <joint name="base_joint" type="fixed">
-    <parent link="world" />
-    <origin xyz="0 0 0" rpy="0 0 0" />
-    <child link="base_link" />
-  </joint>
+<robot xmlns:joint="http://playerstage.sourceforge.net/gazebo/xmlschema/#joint">
   <link name="base_link">
     <inertial>
       <mass value="1000" />
-      <origin xyz=" 0 0 0 " />
+      <origin xyz="0 0 0" rpy="0 0 0"/>
       <inertia ixx="1000" ixy="0" ixz="0" iyy="1000" iyz="0" izz="1000" />
     </inertial>
     <visual>
-      <origin xyz="0 0 0" rpy="0 0 0 " />
-      <geometry name="pr2_base_mesh_file">
+      <origin xyz="0 0 0" rpy="0 0 0" />
+      <geometry>
         <box size=".01 .01 .01" />
       </geometry>
     </visual>
     <collision>
-      <origin xyz="0 0 0" rpy="0.0 0.0 0.0 " />
-      <geometry name="base_collision_geom">
+      <origin xyz="0 0 0" rpy="0.0 0.0 0.0" />
+      <geometry>
         <box size=".01 .01 .01" />
       </geometry>
@@ -31,3 +26,13 @@
     <material>Gazebo/White</material>
   </gazebo>
+  <gazebo>
+    <joint:hinge name="base_fixed_joint">
+      <body1>base_link</body1>
+      <body2>world</body2>
+      <anchor>base_link</anchor>
+      <lowStop>0</lowStop>
+      <highStop>0</highStop>
+      <axis>0 0 1</axis>
+    </joint:hinge>
+  </gazebo>
 </robot>
