Commit message: Added macro for PR2 arm, updated shape of dummy UA in visualizer

File: pr2_component_descriptions/robots/pr2_arm.urdf.xacro (robot description, xacro)
@@ -8,4 +8,7 @@
   <include filename="$(find pr2_description)/urdf/materials.urdf.xacro" />
   <include filename="$(find pr2_description)/urdf/shoulder_v0/shoulder.urdf.xacro" />
+  <include filename="$(find pr2_description)/urdf/upper_arm_v0/upper_arm.urdf.xacro" />
+  <include filename="$(find pr2_description)/urdf/forearm_v0/forearm.urdf.xacro" />
+  <include filename="$(find pr2_description)/urdf/gripper_v0/gripper.urdf.xacro" />
   <include filename="$(find pr2_component_descriptions)/urdf/base_link.urdf.xacro" />
   <!-- generic simulator_gazebo plugins for starting mechanism control, ros time, ros battery -->
@@ -14,34 +17,18 @@
     <origin xyz="0 0 0" rpy="0 0 0" />
   </xacro:pr2_shoulder_v0>
-  <!-- Dummy FA used in burn in test -->
-  <joint name="r_dummy_upper_arm_joint" type="fixed">
-    <axis xyz="0 1 0" />
-    <limit effort="0" velocity="100"/>
-    <safety_controller k_velocity="10" />
-    <dynamics damping="0.0" friction="0.0" />
+  <xacro:pr2_upper_arm_v0 side="r" reflect="-1" parent="r_upper_arm_roll_link"/>
+  <xacro:pr2_forearm_v0 side="r" reflect="-1" parent="r_forearm_roll_link"/>
+  <xacro:pr2_gripper_v0 side="r" parent="r_wrist_roll_link"
+               screw_reduction="${4.0/1000.0}"
+               gear_ratio="${(729.0/25.0)*(22.0/16.0)}"
+               theta0="${3.6029*M_PI/180.0}"
+               phi0="${29.7089*M_PI/180.0}"
+               t0="${-0.1914/1000.0}"
+               L0="${37.5528/1000.0}"
+               h="${0.0/1000.0}"
+               a="${68.3698/1000.0}"
+               b="${43.3849/1000.0}"
+               r="${91.5/1000.0}" >
     <origin xyz="0 0 0" rpy="0 0 0" />
-    <parent link="r_upper_arm_roll_link"/>
-    <child link="r_dummy_upper_arm_link"/>
-  </joint>
-  <link name="r_dummy_upper_arm_link">
-    <inertial>
-      <mass value="1" />
-      <origin xyz=" 0 0 0 " />
-      <inertia  ixx="1.0" ixy="0.0" ixz="0.0"
-                iyy="1.0" iyz="0.0" izz="1.0" />
-    </inertial>
-    <visual>
-      <origin xyz="0.12 0 0" rpy="0 0 0" />
-      <geometry>
-	<box size="0.60 0.06 0.15" />
-      </geometry>
-    </visual>
-  </link>
-<!--
-  <transmission type="SimpleTransmission" name="r_dummy_upperarm_trans">
-    <actuator name="r_elbow_flex_motor" />
-    <joint name="r_dummy_upper_arm_joint" />
-    <mechanicalReduction>1</mechanicalReduction>
-  </transmission>
- -->
+  </xacro:pr2_gripper_v0>
 </robot>

Commit message: Adding origin to forearm macro in pr2_component_descriptions

File: pr2_component_descriptions/robots/pr2_arm.urdf.xacro (robot description, xacro)
@@ -18,5 +18,7 @@
   </xacro:pr2_shoulder_v0>
   <xacro:pr2_upper_arm_v0 side="r" reflect="-1" parent="r_upper_arm_roll_link"/>
-  <xacro:pr2_forearm_v0 side="r" reflect="-1" parent="r_forearm_roll_link"/>
+  <xacro:pr2_forearm_v0 side="r" reflect="-1" parent="r_forearm_roll_link" >
+       <origin xyz="0 0 0" rpy="0 0 0" />
+  </xacro:pr2_forearm_v0>
   <xacro:pr2_gripper_v0 side="r" parent="r_wrist_roll_link"
                screw_reduction="${4.0/1000.0}"

Commit message: Modified pr2_arm URDF to allow random poses controller to work it.

File: pr2_component_descriptions/robots/pr2_arm.urdf.xacro (robot description, xacro)
@@ -14,5 +14,19 @@
   <!-- generic simulator_gazebo plugins for starting mechanism control, ros time, ros battery -->
   <include filename="$(find pr2_description)/gazebo/gazebo.urdf.xacro" />
-  <xacro:pr2_shoulder_v0 side="r" reflect="-1" parent="base_link">
+  <!-- Bogus torso_lift_link for commands to arm -->
+  <joint name="torso_link_joint" type="fixed" >
+    <parent link="base_link" />
+    <child link="torso_lift_link" />
+    <origin xyz="0 0 0" rpy="0 0 0" />
+  </joint>
+  <link name="torso_lift_link">
+    <inertial>
+      <mass value="1" />
+      <origin xyz=" 0 0 0 " />
+      <inertia  ixx="1.0" ixy="0.0" ixz="0.0"
+                iyy="1.0" iyz="0.0" izz="1.0" />
+    </inertial>
+  </link>
+  <xacro:pr2_shoulder_v0 side="r" reflect="-1" parent="torso_lift_link">
     <origin xyz="0 0 0" rpy="0 0 0" />
   </xacro:pr2_shoulder_v0>

Commit message: need visual and collision because it has children.

File: pr2_component_descriptions/robots/pr2_arm.urdf.xacro (robot description, xacro)
@@ -27,4 +27,16 @@
                 iyy="1.0" iyz="0.0" izz="1.0" />
     </inertial>
+    <visual>
+      <origin xyz="0 0 0" rpy="0 0 0" />
+      <geometry>
+        <box size=".01 .01 .01" />
+      </geometry>
+    </visual>
+    <collision>
+      <origin xyz="0 0 0" rpy="0.0 0.0 0.0" />
+      <geometry>
+        <box size=".01 .01 .01" />
+      </geometry>
+    </collision>
   </link>
   <xacro:pr2_shoulder_v0 side="r" reflect="-1" parent="torso_lift_link">

Commit message: raise arm so it's not in collision with ground

File: pr2_component_descriptions/robots/pr2_arm.urdf.xacro (robot description, xacro)
@@ -18,5 +18,5 @@
     <parent link="base_link" />
     <child link="torso_lift_link" />
-    <origin xyz="0 0 0" rpy="0 0 0" />
+    <origin xyz="0 0 1" rpy="0 0 0" />
   </joint>
   <link name="torso_lift_link">
