Commit message: Comitting shoulder dummy upperarm launch file for burn in.

File: pr2_component_descriptions/robots/shoulder_dummy_ua.urdf.xacro (robot description, xacro)
@@ -1,4 +1,4 @@
 <?xml version="1.0"?>
-<robot name="pr2_upper_arm"
+<robot name="shoulder"
        xmlns:sensor="http://playerstage.sourceforge.net/gazebo/xmlschema/#sensor"
        xmlns:controller="http://playerstage.sourceforge.net/gazebo/xmlschema/#controller"
@@ -7,11 +7,13 @@
   <include filename="$(find pr2_description)/urdf/common.xacro" />
   <include filename="$(find pr2_description)/urdf/materials.urdf.xacro" />
-  <include filename="$(find pr2_description)/urdf/upper_arm_v0/upper_arm.urdf.xacro" />
+  <include filename="$(find pr2_description)/urdf/shoulder_v0/shoulder.urdf.xacro" />
   <include filename="$(find pr2_component_descriptions)/urdf/base_link.urdf.xacro" />
-  <xacro:pr2_upper_arm_v0 side="r" reflect="-1" parent="base_link">
+  <!-- generic simulator_gazebo plugins for starting mechanism control, ros time, ros battery -->
+  <include filename="$(find pr2_description)/gazebo/gazebo.urdf.xacro" />
+  <xacro:pr2_shoulder_v0 side="r" reflect="-1" parent="base_link">
     <origin xyz="0 0 0" rpy="0 0 0" />
-  </xacro:pr2_upper_arm_v0>
-    <!-- Dummy FA used in burn in test -->
-  <joint name="r_dummy_forearm_joint" type="fixed">
+  </xacro:pr2_shoulder_v0>
+  <!-- Dummy FA used in burn in test -->
+  <joint name="r_dummy_upper_arm_joint" type="fixed">
     <axis xyz="0 1 0" />
     <limit effort="0" velocity="100"/>
@@ -19,8 +21,8 @@
     <dynamics damping="0.0" friction="0.0" />
     <origin xyz="0 0 0" rpy="0 0 0" />
-    <parent link="r_forearm_roll_link"/>
-    <child link="r_dummy_forearm_link"/>
+    <parent link="r_upper_arm_roll_link"/>
+    <child link="r_dummy_upper_arm_link"/>
   </joint>
-  <link name="r_dummy_forearm_link">
+  <link name="r_dummy_upper_arm_link">
     <inertial>
       <mass value="1" />
@@ -30,14 +32,14 @@
     </inertial>
     <visual>
-      <origin xyz="0.10 0 0" rpy="0 0 0" />
+      <origin xyz="0.12 0 0" rpy="0 0 0" />
       <geometry>
-	<box size="0.25 0.08 0.08" />
+	<box size="0.60 0.015 0.08" />
       </geometry>
     </visual>
   </link>
 <!--
-  <transmission type="SimpleTransmission" name="r_dummy_forearm_trans">
-    <actuator name="r_wrist_l_motor" />
-    <joint name="r_dummy_forearm_joint" />
+  <transmission type="SimpleTransmission" name="r_dummy_upperarm_trans">
+    <actuator name="r_elbow_flex_motor" />
+    <joint name="r_dummy_upper_arm_joint" />
     <mechanicalReduction>1</mechanicalReduction>
   </transmission>

File: pr2_component_descriptions/robots/wrist_gripper.urdf.xacro (robot description, xacro)
@@ -8,5 +8,4 @@
   <include filename="$(find pr2_description)/urdf/materials.urdf.xacro" />
   <include filename="$(find pr2_description)/urdf/forearm_v0/forearm.urdf.xacro" />
-  <include filename="$(find pr2_description)/urdf/gripper_v0/gripper.urdf.xacro" />
   <include filename="$(find pr2_component_descriptions)/urdf/base_link.urdf.xacro" />
    <!-- generic simulator_gazebo plugins for starting mechanism control, ros time, ros battery -->
@@ -16,5 +15,5 @@
   </xacro:pr2_forearm_v0>
   <!-- Dummy gripper used in burn in test -->
-  <joint name="r_gripper_fake_joint" type="continuous">
+  <joint name="r_gripper_fake_joint" type="fixed" >
     <axis xyz="0 1 0" />
     <limit effort="0" velocity="100"/>
@@ -39,9 +38,3 @@
     </visual>
   </link>
-  <!-- Transmission uses r_gripper_motor -->
-  <transmission type="SimpleTransmission" name="r_gripper_fake_trans">
-    <actuator name="r_gripper_motor" />
-    <joint name="r_gripper_fake_joint" />
-    <mechanicalReduction>1</mechanicalReduction>
-  </transmission>
 </robot>

Commit message: Adding features to UA roll URDF used in qual. #3927

File: pr2_component_descriptions/robots/shoulder_dummy_ua.urdf.xacro (robot description, xacro)
@@ -38,10 +38,3 @@
     </visual>
   </link>
-<!--
-  <transmission type="SimpleTransmission" name="r_dummy_upperarm_trans">
-    <actuator name="r_elbow_flex_motor" />
-    <joint name="r_dummy_upper_arm_joint" />
-    <mechanicalReduction>1</mechanicalReduction>
-  </transmission>
- -->
 </robot>

File: pr2_component_descriptions/robots/upper_arm_roll.urdf.xacro (robot description, xacro)
@@ -15,3 +15,27 @@
     <origin xyz="0 0 0" rpy="0 0 0" />
   </xacro:pr2_upper_arm_roll_v0>
+  <!-- Dummy FA used in burn in test -->
+  <joint name="r_dummy_upper_arm_joint" type="fixed">
+    <axis xyz="0 1 0" />
+    <limit effort="0" velocity="100"/>
+    <safety_controller k_velocity="10" />
+    <dynamics damping="0.0" friction="0.0" />
+    <origin xyz="0 0 0" rpy="0 0 0" />
+    <parent link="r_upper_arm_roll_link"/>
+    <child link="r_dummy_upper_arm_link"/>
+  </joint>
+  <link name="r_dummy_upper_arm_link">
+    <inertial>
+      <mass value="1" />
+      <origin xyz=" 0 0 0 " />
+      <inertia  ixx="1.0" ixy="0.0" ixz="0.0"
+                iyy="1.0" iyz="0.0" izz="1.0" />
+    </inertial>
+    <visual>
+      <origin xyz="0.12 0 0" rpy="0 0 0" />
+      <geometry>
+	<box size="0.10 0.06 0.15" />
+      </geometry>
+    </visual>
+  </link>
 </robot>
