Commit message: Added links to urdf to make pr2_etherCAT happy. Added delay to projector monitor to avoid catching error occuring during pr2_etherCAT startup.

File: qualification/tests/projector_test/robot.urdf (robot description, URDF)
Before this commit: robot robot_none, 1 links, 0 joints
Links:
- removed link there_are_no_links_for_this_test
- added link there-is-no-need-for-any-links-on-a-projector
Joints:
- added joint no-joints-either: type continuous, parent world, child there-is-no-need-for-any-links-on-a-projector

Commit message: Gripper tip test is tested on actual tip, just needs to get SN worked out. Shoulder, UA, Full arm cameras now run on eth2

File: qualification/tests/projector_test/robot.urdf (robot description, URDF)
Before this commit: robot robot_none, 1 links, 1 joints
Links:
- removed link there-is-no-need-for-any-links-on-a-projector
- added link there_are_no_links_for_this_test, mass 1
Joints:
- removed joint no-joints-either
